File: sq_lockin_v8/2opamp.kicad_sch (KiCad schematic)
At the start: 2 parts

Commit message: Keep boards up to date
Parts:
- U11: Field5 (none) -> C46316 / OPA2376; LCSC C46316 -> C1517414; MPN OPA2376AIDR -> OPA2388IDR
Changed lines of the file:
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@@
       (effects (font (size 1.27 1.27)) hide)
     )
-    (property "LCSC" "C46316" (id 4) (at 120.65 133.35 0)
+    (property "LCSC" "C1517414" (id 4) (at 120.65 133.35 0)
       (effects (font (size 1.27 1.27)) hide)
     )
-    (property "MPN" "OPA2376AIDR" (id 5) (at 120.65 133.35 0)
+    (property "MPN" "OPA2388IDR" (id 5) (at 120.65 133.35 0)
+      (effects (font (size 1.27 1.27)) hide)
+    )
+    (property "Field5" "C46316 / OPA2376" (id 6) (at 120.65 133.35 0)
       (effects (font (size 1.27 1.27)) hide)
     )
@@
       (effects (font (size 1.27 1.27)) hide)
     )
-    (property "LCSC" "C46316" (id 4) (at 120.65 101.6 0)
+    (property "LCSC" "C1517414" (id 4) (at 120.65 101.6 0)
       (effects (font (size 1.27 1.27)) hide)
     )
-    (property "MPN" "OPA2376AIDR" (id 5) (at 120.65 101.6 0)
+    (property "MPN" "OPA2388IDR" (id 5) (at 120.65 101.6 0)
+      (effects (font (size 1.27 1.27)) hide)
+    )
+    (property "Field5" "C46316 / OPA2376" (id 6) (at 120.65 101.6 0)
       (effects (font (size 1.27 1.27)) hide)
     )
@@
       (effects (font (size 1.27 1.27)) hide)
     )
-    (property "LCSC" "C46316" (id 4) (at 207.01 118.11 0)
+    (property "LCSC" "C1517414" (id 4) (at 207.01 118.11 0)
       (effects (font (size 1.27 1.27)) hide)
     )
-    (property "MPN" "OPA2376AIDR" (id 5) (at 207.01 118.11 0)
+    (property "MPN" "OPA2388IDR" (id 5) (at 207.01 118.11 0)
       (effects (font (size 1.27 1.27)) hide)
     )
+    (property "Field5" "C46316 / OPA2376" (id 6) (at 207.01 118.11 0)
+      (effects (font (size 1.27 1.27)) hide)
+    )
