File: sq_lockin_v8/IA.kicad_sch (KiCad schematic)
At the start: 11 parts

Commit message: Keep boards up to date
Parts:
- added C19, C20: (no value), symbol 0JLC-6:10uF_1206_50V
- added JP1: (no value), symbol Jumper:Jumper_2_Open
- added R11: (no value), symbol 0JLC-6:100
- added R12: (no value), symbol 0JLC-6:2K
- U12: Field5 (none) -> C46316 / OPA2376; LCSC C46316 -> C1517414; MPN OPA2376AIDR -> OPA2388IDR
- renumbered C19 to C21, R11 to R13, R12 to R14
Connections:
- net GND: now also C19.2
- net at R10.1, U14.1, U14.4 (-): now also C20.1
- net at R13.2, R14.1: now also R12.2; no longer U14.3 (+)
- new net: C19.1, R11.1, U14.3 (+)
- new net: C20.2, JP1.1 (A)
- new net: JP1.2 (B), R11.2, R12.1
Other:
- moved on the sheet: C21, R13, R14
