File: sq_lockin_v8/hx710c.kicad_sch (KiCad schematic)
At the start: 6 parts

Commit message: Keep boards up to date
Parts:
- renumbered C20 to C22, C21 to C23, C22 to C24, R13 to R15, R14 to R16
Changed lines of the file:
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@@
   (symbol (lib_id "power:GND") (at 137.16 85.09 270) (unit 1)
     (in_bom yes) (on_board yes)
-    (property "Reference" "#PWR050" (id 0) (at 130.81 85.09 0)
+    (property "Reference" "#PWR051" (id 0) (at 130.81 85.09 0)
       (effects (font (size 1.27 1.27)) hide)
     )
@@
   (symbol (lib_id "0JLC-6:100nF") (at 129.54 92.71 180) (unit 1)
     (in_bom yes) (on_board yes)
-    (property "Reference" "C20" (id 0) (at 132.461 91.5416 0)
+    (property "Reference" "C22" (id 0) (at 132.461 91.5416 0)
       (effects (font (size 1.27 1.27)) (justify right))
     )
@@
   (symbol (lib_id "0JLC-6:10") (at 125.73 87.63 270) (unit 1)
     (in_bom yes) (on_board yes)
-    (property "Reference" "R13" (id 0) (at 125.73 82.3722 90))
+    (property "Reference" "R15" (id 0) (at 125.73 82.3722 90))
     (property "Value" "" (id 1) (at 125.73 84.6836 90))
     (property "Footprint" "" (id 2) (at 125.73 85.852 90)
@@
   (symbol (lib_id "0JLC-6:10") (at 125.73 96.52 270) (unit 1)
     (in_bom yes) (on_board yes)
-    (property "Reference" "R14" (id 0) (at 125.73 91.2622 90))
+    (property "Reference" "R16" (id 0) (at 125.73 91.2622 90))
     (property "Value" "" (id 1) (at 125.73 93.5736 90))
     (property "Footprint" "" (id 2) (at 125.73 94.742 90)
@@
   (symbol (lib_id "0JLC-6:100nF") (at 132.08 77.47 270) (unit 1)
     (in_bom yes) (on_board yes)
-    (property "Reference" "C21" (id 0) (at 132.08 71.0692 90))
+    (property "Reference" "C23" (id 0) (at 132.08 71.0692 90))
     (property "Value" "" (id 1) (at 132.08 73.3806 90))
     (property "Footprint" "" (id 2) (at 128.27 78.4352 0)
@@
   (symbol (lib_id "power:GND") (at 128.27 77.47 270) (unit 1)
     (in_bom yes) (on_board yes)
-    (property "Reference" "#PWR049" (id 0) (at 121.92 77.47 0)
+    (property "Reference" "#PWR050" (id 0) (at 121.92 77.47 0)
       (effects (font (size 1.27 1.27)) hide)
     )
@@
   (symbol (lib_id "0JLC-6:100nF") (at 157.48 73.66 90) (mirror x) (unit 1)
     (in_bom yes) (on_board yes)
-    (property "Reference" "C22" (id 0) (at 157.48 67.2592 90))
+    (property "Reference" "C24" (id 0) (at 157.48 67.2592 90))
     (property "Value" "" (id 1) (at 157.48 69.5706 90))
     (property "Footprint" "" (id 2) (at 161.29 74.6252 0)
@@
   (symbol (lib_id "power:GND") (at 153.67 73.66 270) (mirror x) (unit 1)
     (in_bom yes) (on_board yes)
-    (property "Reference" "#PWR051" (id 0) (at 147.32 73.66 0)
+    (property "Reference" "#PWR052" (id 0) (at 147.32 73.66 0)
       (effects (font (size 1.27 1.27)) hide)
     )
@@
   (symbol (lib_id "power:VCC") (at 163.83 85.09 0) (unit 1)
     (in_bom yes) (on_board yes)
-    (property "Reference" "#PWR052" (id 0) (at 163.83 88.9 0)
+    (property "Reference" "#PWR053" (id 0) (at 163.83 88.9 0)
       (effects (font (size 1.27 1.27)) hide)
     )
