File: sq_lockin_v8/power.kicad_sch (KiCad schematic)
At the start: 30 parts

Commit message: Keep boards up to date
Parts:
- D6: value LBAT54HT1G -> (none); footprint Diode_SMD:D_SOD-323 -> (none)
- renumbered C26 to C28, C27 to C29, C28 to C30, C29 to C31, C30 to C32, C31 to C33, C32 to C34, C33 to C35, C34 to C36, C35 to C37, C36 to C38, C37 to C39, R17 to R19, R18 to R20
Connections:
- net Vd: now also C29.1, C30.1, D4.1 (K), D5.1 (K), L1.2, L2.2; no longer C31.1, D4.2 (A), U17.5 (OUT)
- new net: C31.1, D4.2 (A), U17.5 (OUT)
Changed lines of the file:
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@@
   (junction (at 66.04 143.51) (diameter 0) (color 0 0 0 0)
   )
+  (junction (at 64.77 95.25) (diameter 0) (color 0 0 0 0)
+  )
   (junction (at 172.72 110.49) (diameter 0) (color 0 0 0 0)
   )
@@
   )
   (wire (pts (xy 58.42 68.58) (xy 62.23 68.58))
+    (stroke (width 0) (type default) (color 0 0 0 0))
+  )
+  (wire (pts (xy 64.77 95.25) (xy 66.548 95.25))
     (stroke (width 0) (type default) (color 0 0 0 0))
   )
@@
     (effects (font (size 1.27 1.27)) (justify right))
   )
-  (hierarchical_label "Vd" (shape output) (at 95.25 68.58 0)
+  (hierarchical_label "Vd" (shape output) (at 66.548 95.25 0)
     (effects (font (size 1.27 1.27)) (justify left))
   )
@@
   (symbol (lib_id "0JLC-6:100nF") (at 129.54 105.41 180) (unit 1)
     (in_bom yes) (on_board yes)
-    (property "Reference" "C32" (id 0) (at 128.905 107.95 0)
+    (property "Reference" "C34" (id 0) (at 128.905 107.95 0)
       (effects (font (size 1.27 1.27)) (justify left))
     )
@@
   (symbol (lib_id "Device:C") (at 144.78 105.41 180) (unit 1)
     (in_bom yes) (on_board yes)
-    (property "Reference" "C34" (id 0) (at 144.145 107.95 0)
+    (property "Reference" "C36" (id 0) (at 144.145 107.95 0)
       (effects (font (size 1.27 1.27)) (justify left))
     )
@@
   (symbol (lib_id "power:GND") (at 144.78 111.76 0) (unit 1)
     (in_bom yes) (on_board yes)
-    (property "Reference" "#PWR057" (id 0) (at 144.78 118.11 0)
+    (property "Reference" "#PWR058" (id 0) (at 144.78 118.11 0)
       (effects (font (size 1.27 1.27)) hide)
     )
@@
   (symbol (lib_id "power:GND") (at 172.72 119.38 0) (unit 1)
     (in_bom yes) (on_board yes)
-    (property "Reference" "#PWR059" (id 0) (at 172.72 125.73 0)
+    (property "Reference" "#PWR060" (id 0) (at 172.72 125.73 0)
       (effects (font (size 1.27 1.27)) hide)
     )
@@
   (symbol (lib_id "0JLC-6:10uF_1206_50V") (at 113.03 105.41 0) (unit 1)
     (in_bom yes) (on_board yes)
-    (property "Reference" "C30" (id 0) (at 115.57 106.68 0)
+    (property "Reference" "C32" (id 0) (at 115.57 106.68 0)
       (effects (font (size 1.27 1.27)) (justify left))
     )
@@
   (symbol (lib_id "0JLC-6:4.7uF_1206_50V") (at 64.77 105.41 0) (unit 1)
     (in_bom yes) (on_board yes)
-    (property "Reference" "C27" (id 0) (at 67.691 104.2416 0)
+    (property "Reference" "C29" (id 0) (at 67.691 104.2416 0)
       (effects (font (size 1.27 1.27)) (justify left))
     )
@@
   (symbol (lib_id "0JLC-6:1K") (at 172.72 105.41 0) (unit 1)
     (in_bom yes) (on_board yes)
-    (property "Reference" "R17" (id 0) (at 174.498 104.2416 0)
+    (property "Reference" "R19" (id 0) (at 174.498 104.2416 0)
       (effects (font (size 1.27 1.27)) (justify left))
     )
@@
   (symbol (lib_id "Device:C") (at 172.72 115.57 0) (unit 1)
     (in_bom yes) (on_board yes)
-    (property "Reference" "C36" (id 0) (at 175.641 114.4016 0)
+    (property "Reference" "C38" (id 0) (at 175.641 114.4016 0)
       (effects (font (size 1.27 1.27)) (justify left))
     )
@@
   (symbol (lib_id "Device:C") (at 146.05 137.16 180) (unit 1)
     (in_bom yes) (on_board yes)
-    (property "Reference" "C35" (id 0) (at 145.415 139.7 0)
+    (property "Reference" "C37" (id 0) (at 145.415 139.7 0)
       (effects (font (size 1.27 1.27)) (justify left))
     )
@@
   (symbol (lib_id "power:GND") (at 214.63 119.38 0) (unit 1)
     (in_bom yes) (on_board yes)
-    (property "Reference" "#PWR061" (id 0) (at 214.63 125.73 0)
+    (property "Reference" "#PWR062" (id 0) (at 214.63 125.73 0)
       (effects (font (size 1.27 1.27)) hide)
     )
@@
   (symbol (lib_id "power:GND") (at 248.92 119.38 0) (unit 1)
     (in_bom yes) (on_board yes) (fields_autoplaced)
-    (property "Reference" "#PWR062" (id 0) (at 248.92 125.73 0)
+    (property "Reference" "#PWR063" (id 0) (at 248.92 125.73 0)
       (effects (font (size 1.27 1.27)) hide)
     )
@@
   (symbol (lib_id "0JLC-6:100nF") (at 130.81 137.16 180) (unit 1)
     (in_bom yes) (on_board yes)
-    (property "Reference" "C33" (id 0) (at 130.175 139.7 0)
+    (property "Reference" "C35" (id 0) (at 130.175 139.7 0)
       (effects (font (size 1.27 1.27)) (justify left))
     )
@@
   (symbol (lib_id "0JLC-6:4.7uF_1206_50V") (at 66.04 137.16 0) (unit 1)
     (in_bom yes) (on_board yes)
-    (property "Reference" "C28" (id 0) (at 68.961 135.9916 0)
+    (property "Reference" "C30" (id 0) (at 68.961 135.9916 0)
       (effects (font (size 1.27 1.27)) (justify left))
     )
@@
   (symbol (lib_id "0JLC-6:1uF") (at 85.09 72.39 0) (unit 1)
     (in_bom yes) (on_board yes)
-    (property "Reference" "C29" (id 0) (at 88.011 71.2216 0)
+    (property "Reference" "C31" (id 0) (at 88.011 71.2216 0)
       (effects (font (size 1.27 1.27)) (justify left))
     )
@@
   (symbol (lib_id "power:GND") (at 199.39 119.38 0) (unit 1)
     (in_bom yes) (on_board yes) (fields_autoplaced)
-    (property "Reference" "#PWR060" (id 0) (at 199.39 125.73 0)
+    (property "Reference" "#PWR061" (id 0) (at 199.39 125.73 0)
       (effects (font (size 1.27 1.27)) hide)
     )
@@
   (symbol (lib_id "0JLC-6:1K") (at 214.63 105.41 0) (unit 1)
     (in_bom yes) (on_board yes)
-    (property "Reference" "R18" (id 0) (at 216.408 104.2416 0)
+    (property "Reference" "R20" (id 0) (at 216.408 104.2416 0)
       (effects (font (size 1.27 1.27)) (justify left))
     )
@@
   (symbol (lib_id "0JLC-6:10uF_1206_50V") (at 114.3 137.16 0) (unit 1)
     (in_bom yes) (on_board yes)
-    (property "Reference" "C31" (id 0) (at 116.84 138.43 0)
+    (property "Reference" "C33" (id 0) (at 116.84 138.43 0)
       (effects (font (size 1.27 1.27)) (justify left))
     )
@@
     (in_bom yes) (on_board yes)
     (property "Reference" "D6" (id 0) (at 50.8 44.45 90))
-    (property "Value" "LBAT54HT1G" (id 1) (at 54.61 46.99 90))
-    (property "Footprint" "Diode_SMD:D_SOD-323" (id 2) (at 43.18 45.72 0)
+    (property "Value" "" (id 1) (at 54.61 46.99 90))
+    (property "Footprint" "" (id 2) (at 43.18 45.72 0)
       (effects (font (size 1.27 1.27)) hide)
     )
@@
   (symbol (lib_id "power:GNDD") (at 157.48 140.97 0) (unit 1)
     (in_bom yes) (on_board yes) (fields_autoplaced)
-    (property "Reference" "#PWR058" (id 0) (at 157.48 147.32 0)
+    (property "Reference" "#PWR059" (id 0) (at 157.48 147.32 0)
       (effects (font (size 1.27 1.27)) hide)
     )
@@
   (symbol (lib_id "Device:C") (at 214.63 115.57 0) (unit 1)
     (in_bom yes) (on_board yes)
-    (property "Reference" "C37" (id 0) (at 217.551 114.4016 0)
+    (property "Reference" "C39" (id 0) (at 217.551 114.4016 0)
       (effects (font (size 1.27 1.27)) (justify left))
     )
@@
   (symbol (lib_id "0JLC-6:1uF") (at 58.42 72.39 0) (unit 1)
     (in_bom yes) (on_board yes)
-    (property "Reference" "C26" (id 0) (at 61.341 71.2216 0)
-      (effects (font (size 1.27 1.27)) (justify left))
-    )
+    (property "Reference" "C28" (id 0) (at 61.341 71.2216 0)
+      (effects (font (size 1.27 1.27)) (justify left))
+    )
