File: sq_lockin_v8/sq_lockin_v8.kicad_pcb (KiCad board)
At the start: 2 copper layers, 125 x 70 mm, 102 parts, among them J1 Conn_01x04, J10 battery, J11 battery, J12 Conn_Coaxial, J13 Conn_Coaxial, J2 Conn_01x02_Male_2.54mm, J3 Conn_01x02_Male_2.54mm, J4 Conn_01x02_Male_2.54mm, J5 battery, J6 Conn_01x02_Male_2.54mm, J7 Conn_Coaxial, J8 JST_SH_Conn_01x04_i2c_horizon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, J9 USB_C_KoreanHroparts_6P, Q1 BC847C, Q2 FZT851TA, U1 NC7SB3157P6X, U10 RS2105XN, U11 OPA2376xxDGK, U12 OPA2376xxDGK, U13 INA826, U14 OPA333xxDBV, U15 HX710C, U16 HX710C, U17 LP5907MFX-3.3, U2 LP5907MFX-3.3, U3 REF3325, U4 pi162U, U5 seeed_rp2040, U6 PI121, U7 pi142M31, U8 RS2105XN, U9 RS2105XN

Commit message: Keep boards up to date
Parts:
- added C19: 10uF, Capacitor_SMD:C_1210_3225Metric_Pad1.33x2.70mm_HandSolder, F.Cu at (156.4, 102.7)
- added C20: 47uF, Capacitor_SMD:C_1210_3225Metric_Pad1.33x2.70mm_HandSolder, F.Cu at (157.7, 108.9)
- added JP1: Jumper_2_Open, Jumper:SolderJumper-2_P1.3mm_Open_RoundedPad1.0x1.5mm, F.Cu at (153.2, 108.5)
- added R11: 100, Resistor_SMD:R_0603_1608Metric_Pad0.98x0.95mm_HandSolder, F.Cu at (153.9, 101.9)
- added R12: 2K, Resistor_SMD:R_0603_1608Metric_Pad0.98x0.95mm_HandSolder, F.Cu at (152.2, 101.9)
- C12, C13, C14: footprint Capacitor_SMD:C_0402_1005Metric -> Capacitor_SMD:C_0402_1005Metric_Pad0.74x0.62mm_HandSolder
- C2, C3, C4, C6: footprint Capacitor_SMD:C_0603_1608Metric_Pad1.05x0.95mm_HandSolder -> Capacitor_SMD:C_0603_1608Metric_Pad1.08x0.95mm_HandSolder
- C21: renamed from C19; value 100nF -> 100nF_0402; footprint Capacitor_SMD:C_0603_1608Metric_Pad1.08x0.95mm_HandSolder -> Capacitor_SMD:C_0402_1005Metric
- R13: renamed from R11; value 10K -> 1K; footprint Resistor_SMD:R_0603_1608Metric_Pad1.05x0.95mm_HandSolder -> Resistor_SMD:R_0402_1005Metric_Pad0.72x0.64mm_HandSolder
- R14: renamed from R12; value 10K -> 1K; footprint Resistor_SMD:R_0603_1608Metric_Pad1.05x0.95mm_HandSolder -> Resistor_SMD:R_0402_1005Metric_Pad0.72x0.64mm_HandSolder
- R15: renamed from R13; footprint Resistor_SMD:R_0603_1608Metric_Pad1.05x0.95mm_HandSolder -> Resistor_SMD:R_0603_1608Metric_Pad0.98x0.95mm_HandSolder
- R16: renamed from R14; footprint Resistor_SMD:R_0603_1608Metric_Pad1.05x0.95mm_HandSolder -> Resistor_SMD:R_0603_1608Metric_Pad0.98x0.95mm_HandSolder
- R17: renamed from R15; footprint Resistor_SMD:R_0603_1608Metric_Pad1.05x0.95mm_HandSolder -> Resistor_SMD:R_0603_1608Metric_Pad0.98x0.95mm_HandSolder
- R18: renamed from R16; footprint Resistor_SMD:R_0603_1608Metric_Pad1.05x0.95mm_HandSolder -> Resistor_SMD:R_0603_1608Metric_Pad0.98x0.95mm_HandSolder
- U11, U12: value OPA2376xxDGK -> OPA2388
- U14: value OPA333xxDBV -> OPA388
- moved C21 5.92 mm to (152.5, 96.8), turned to 180 degrees
- moved R14 5.66 mm to (153.1, 98.7), turned to 90 degrees
- moved R13 5.24 mm to (151.9, 98.7)
- moved J9 0.09 mm to (200.2, 112.5)
- renumbered C20 to C22, C21 to C23, C22 to C24, C23 to C25, C24 to C26, C25 to C27, C26 to C28, C27 to C29, C28 to C30, C29 to C31, C30 to C32, C31 to C33, C32 to C34, C33 to C35, C34 to C36, C35 to C37, C36 to C38, C37 to C39, R17 to R19, R18 to R20
Connections:
- C29 pad 1: Net-(C27-Pad1) -> VD
- C30 pad 1: Net-(C27-Pad1) -> VD
- C31 pad 1: VD -> Net-(C31-Pad1)
- D4 pad 1: Net-(C27-Pad1) -> VD
- D4 pad 2: VD -> Net-(C31-Pad1)
- D5 pad 1: Net-(C27-Pad1) -> VD
- L1 pad 2: Net-(C27-Pad1) -> VD
- L2 pad 2: Net-(C27-Pad1) -> VD
- R13 pad 2: Net-(R11-Pad2) -> Net-(R12-Pad2)
- R14 pad 1: Net-(R11-Pad2) -> Net-(R12-Pad2)
- U14 pad 3: Net-(R11-Pad2) -> Net-(C19-Pad1)
- U17 pad 5: VD -> Net-(C31-Pad1)
Routing:
- net VD: track 14.2 -> 103.6 mm, vias 0 -> 2
- net Net-(C27-Pad1): track 87.3 -> 0.00 mm, vias 2 -> 0
- net /vref: track 95.0 -> 83.5 mm, vias 5 -> 6
- net Net-(JP1-Pad2): track 0.00 -> 8.99 mm, vias 0 -> 2
- net Net-(C20-Pad1): track 10.0 -> 17.4 mm, vias 0 -> 2
- net Net-(C19-Pad1): track 0.00 -> 4.84 mm
- net Net-(C31-Pad1): track 0.00 -> 4.33 mm
- net Net-(R11-Pad2): track 4.20 -> 0.00 mm
- net Net-(R12-Pad2): track 0.00 -> 3.03 mm
- net Net-(C20-Pad2): track 0.00 -> 2.45 mm
- net GND: track 76.3 -> 75.1 mm, vias 12 -> 13
- net +3V3: track 221.8 -> 222.6 mm
Other:
- board text added: "sq_lockin_v8B 4/2023"
- board text removed: "sq_lockin_v8 9/2022"
