File: level_translator/power.kicad_sch (KiCad schematic)
At the start: 7 parts

Commit message: Add tweaks to diode readout
Parts:
- U2: value ~ -> (none); footprint Package_TO_SOT_SMD:SOT-23-5 -> (none); LCSC C80670 -> C529554; MPN LP5907MFX-3.3/NOPB -> LP5907MFX-4.5/NOPB
Changed lines of the file:
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@@
     (in_bom yes) (on_board yes)
     (property "Reference" "U2" (id 0) (at 199.39 84.6582 0))
-    (property "Value" "~" (id 1) (at 199.39 86.9696 0))
-    (property "Footprint" "Package_TO_SOT_SMD:SOT-23-5" (id 2) (at 199.39 85.09 0)
+    (property "Value" "" (id 1) (at 199.39 86.9696 0))
+    (property "Footprint" "" (id 2) (at 199.39 85.09 0)
       (effects (font (size 1.27 1.27)) hide)
     )
@@
       (effects (font (size 1.27 1.27)) hide)
     )
-    (property "LCSC" "C80670" (id 4) (at 199.39 93.98 0)
+    (property "LCSC" "C529554" (id 4) (at 199.39 93.98 0)
       (effects (font (size 1.27 1.27)) hide)
     )
-    (property "MPN" "LP5907MFX-3.3/NOPB" (id 5) (at 199.39 93.98 0)
+    (property "MPN" "LP5907MFX-4.5/NOPB" (id 5) (at 199.39 93.98 0)
       (effects (font (size 1.27 1.27)) hide)
     )
